Commit message: Modify the tf so that camera is linked with camera_link

File: simulation_tobot/URDF/tobot.urdf.xacro (robot description, xacro)
@@ -157,8 +157,8 @@
   </joint>
   <!--CAMERA-->
-  <link name="camera">
+  <link name="camera_link">
     <visual>
       <geometry>
-        <box size="0.15 .05 .05"/>
+        <box size="0.15 .05 .1865"/>
       </geometry>
       <origin rpy="0 0 0" xyz="0 0 0"/>
@@ -168,5 +168,5 @@
   <joint name="camera" type="fixed">
     <parent link="base_link"/>
-    <child link="camera"/>
+    <child link="camera_link"/>
     <origin xyz="${width} 0 ${GROUND_CLEARANCE-bodylen+posz_camera} " rpy="${-PI/2} 0 ${-PI/2}"/>
   </joint>

Commit message: Modified the yaw pitch yaw of camera joint relative to base_link

File: simulation_tobot/URDF/tobot.urdf.xacro (robot description, xacro)
@@ -169,5 +169,5 @@
     <parent link="base_link"/>
     <child link="camera_link"/>
-    <origin xyz="${width} 0 ${GROUND_CLEARANCE-bodylen+posz_camera} " rpy="${-PI/2} 0 ${-PI/2}"/>
+    <origin xyz="${width} 0 ${GROUND_CLEARANCE-bodylen+posz_camera} " rpy="0 0 0"/>
   </joint>
 </robot>
