Commit message: re-adjust <transmission> tag

File: simulation_tobot/URDF/beebot.xacro (robot description, xacro)
@@ -261,3 +261,22 @@
     <origin xyz="${width + 0.07} 0 0.05 " rpy="0 0 0"/>
   </joint>
+  <!--Transmissions for active wheels-->
+    <!-- Transmission is important to link the joints and the controller -->
+    <transmission name="base_to_lwheel_joint_trans">
+      <type>transmission_interface/SimpleTransmission</type>
+      <joint name="base_to_lwheel" />
+      <actuator name="base_to_lwheel_joint_motor">
+        <hardwareInterface>EffortJointInterface</hardwareInterface>
+        <mechanicalReduction>1</mechanicalReduction>
+      </actuator>
+    </transmission>
+    <transmission name="base_to_rwheel_joint_trans">
+      <type>transmission_interface/SimpleTransmission</type>
+      <joint name="base_to_rwheel" />
+      <actuator name="base_to_rwheel_joint_motor">
+        <hardwareInterface>EffortJointInterface</hardwareInterface>
+        <mechanicalReduction>1</mechanicalReduction>
+      </actuator>
+    </transmission>
 </robot>
+</robot>
