Commit message: modify inertia tag

File: simulation_tobot/URDF/my_simple_test.xacro (robot description, xacro)
@@ -12,10 +12,16 @@
     <material name="blue"/>
   </visual>
+  <collision>
+    <geometry>
+      <cylinder length="2" radius="0.5"/>
+    </geometry>
+  <origin rpy="0 0 0" xyz="0 0 0"/>
+  </collision>
   <inertial>
     <mass value="1"/>
     <origin pry="0 0 0" xyz="0 0 0"/>
-    <inertia ixx="0.1" ixy="0" ixz="0"
-             iyy="0.1" iyz="0"
-             izz="0.01"/>
+    <inertia ixx="1.0" ixy="0" ixz="0"
+             iyy="1.0" iyz="0"
+             izz="1.0"/>
   </inertial>
 </link>
