Commit message: change the height of the camera in urdf file

File: mobile_safeguard_primitive/launch/rtabmapping/tf_config/my_tobot.urdf.xacro (robot description, xacro)
@@ -170,5 +170,5 @@
     <child link="camera_link"/>
     <!--<origin xyz="${width} 0 ${GROUND_CLEARANCE-bodylen+posz_camera} " rpy="0 0 0"/>-->
-    <origin xyz="${width} 0 1.55 " rpy="0 0 0"/>
+    <origin xyz="${width} 0 1.30 " rpy="0 0 0"/>
   </joint>
 </robot>

Commit message: adjust frame tree for actual navigation implementation

File: mobile_safeguard_primitive/launch/rtabmapping/tf_config/my_tobot.urdf.xacro (robot description, xacro)
@@ -14,4 +14,5 @@
   <xacro:property name="fwheel_rad" value="0.0325" />
   <xacro:property name="PI" value="3.1415" />
+  <property name="base_z_origin_to_wheel_origin" value="0.0" />
   <material name="black">
     <color rgba="0 0 0 1"/>
@@ -21,4 +22,22 @@
   </material>
   <!-- Actual frame and materials -->
+  <!-- BASE-FOOTPRINT -->
+  <!-- base_footprint is a fictitious link(frame) that is on the ground right below base_link origin -->
+<!--
+  <link name="base_footprint">
+    <visual>
+        <origin xyz="0 0 0" rpy="0 0 0" />
+        <geometry>
+            <box size="0.001 0.001 0.001" />
+        </geometry>
+    </visual>
+  </link>
+  <joint name="base_footprint_joint" type="fixed">
+  <origin xyz="0 0 ${wheel_rad - base_z_origin_to_wheel_origin}" rpy="0 0 0" />
+    <parent link="base_footprint"/>
+    <child link="base_link" />
+  </joint>
+-->
+  <!-- BASE LINK -->
   <link name="base_link">
     <visual>
